File: Rapid_Prototype_Schematic.sch (EAGLE design)
At the start: 177 parts, among them IC2 SI4459ADY-T1-GE3, IC8 SI4485DY-T1-GE3, J1 XT60-M, J10 XT60-M, J2 XT60-M, J3 Vertical Qwiic Connector, J4 UJ2-MIBH-2-SMT-TR-67, J5 XT60-M, J6 XT60-M, J7 XT60-M, J8 XT60-M, J9 XT60-M, Q1 LTV-8141S, Q10 SI4435DDY, Q11 DMN65D8LFB-7, Q12 SI4435DDY, Q13 DMN65D8LFB-7, Q14 SI4435DDY, Q15 DMN65D8LFB-7, Q16 2N7002PW, Q2 2N7002PW, Q3 DMN65D8LFB-7, Q4 SI4435DDY, Q5 DMN65D8LFB-7, Q6 SI4435DDY, Q7 DMN65D8LFB-7, Q8 SI4435DDY, Q9 DMN65D8LFB-7, U1 LM35DM, U2 LM2904ITPX/NOPB, U3 LM2904ITPX/NOPB, U4 LM2904ITPX/NOPB, U5 LM2904ITPX/NOPB, U6 LM2904ITPX/NOPB, U7 TLV1117LV33DCYR, U8 LT1374IS8-5PBF

Commit message: Resistor value change
Changed the values for the resistors. Increased the size of resistors R25 and R26.
Parts:
- removed R25: 0.005Ω 1%, adafruit:R-US_R1206
- added R67: 0.8Ω 1%, rcl:R-US_R2512
- R13, R14, R20: value 0.005 -> 0.003
- R19: value 0.010Ω -> 0.003Ω
- R26: value 0.005Ω 1% -> 0.8Ω 1%; device adafruit:R-US_R1206 -> rcl:R-US_R2512
Connections:
- net COMBINED_POWER: now also R67.2; no longer R25.2
- net ESC_POWER2: now also R67.1; no longer R25.1
Changed lines of the file:
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@@
 <parts>
 <part name="FRAME3" library="frames" library_urn="urn:adsk.eagle:library:229" deviceset="TABL_L" device="" value="Null Value"/>
-<part name="R14" library="adafruit" library_urn="urn:adsk.eagle:library:420" deviceset="R-US_" device="R1206" package3d_urn="urn:adsk.eagle:package:6240569/1" value="0.005"/>
+<part name="R14" library="adafruit" library_urn="urn:adsk.eagle:library:420" deviceset="R-US_" device="R1206" package3d_urn="urn:adsk.eagle:package:6240569/1" value="0.003"/>
 <part name="R8" library="adafruit" library_urn="urn:adsk.eagle:library:420" deviceset="R-US_" device="R0603" package3d_urn="urn:adsk.eagle:package:6240565/1" value="3.3k"/>
 <part name="C2" library="adafruit" library_urn="urn:adsk.eagle:library:420" deviceset="C-US" device="C0603" package3d_urn="urn:adsk.eagle:package:6240338/1" value="0.1µF"/>
@@
 <part name="C6" library="adafruit" library_urn="urn:adsk.eagle:library:420" deviceset="C-US" device="C0603" package3d_urn="urn:adsk.eagle:package:6240338/1" value="1µF"/>
 <part name="GND31" library="SparkFun-PowerSymbols" deviceset="GND" device=""/>
-<part name="R20" library="adafruit" library_urn="urn:adsk.eagle:library:420" deviceset="R-US_" device="R1206" package3d_urn="urn:adsk.eagle:package:6240569/1" value="0.005"/>
+<part name="R20" library="adafruit" library_urn="urn:adsk.eagle:library:420" deviceset="R-US_" device="R1206" package3d_urn="urn:adsk.eagle:package:6240569/1" value="0.003"/>
 <part name="R16" library="adafruit" library_urn="urn:adsk.eagle:library:420" deviceset="R-US_" device="R0603" package3d_urn="urn:adsk.eagle:package:6240565/1" value="3.3k"/>
 <part name="C12" library="adafruit" library_urn="urn:adsk.eagle:library:420" deviceset="C-US" device="C0603" package3d_urn="urn:adsk.eagle:package:6240338/1" value="0.1µF"/>
@@
 <part name="C15" library="adafruit" library_urn="urn:adsk.eagle:library:420" deviceset="C-US" device="C0603" package3d_urn="urn:adsk.eagle:package:6240338/1" value="1µF"/>
 <part name="GND36" library="SparkFun-PowerSymbols" deviceset="GND" device=""/>
-<part name="R13" library="adafruit" library_urn="urn:adsk.eagle:library:420" deviceset="R-US_" device="R1206" package3d_urn="urn:adsk.eagle:package:6240569/1" value="0.005"/>
+<part name="R13" library="adafruit" library_urn="urn:adsk.eagle:library:420" deviceset="R-US_" device="R1206" package3d_urn="urn:adsk.eagle:package:6240569/1" value="0.003"/>
 <part name="R7" library="adafruit" library_urn="urn:adsk.eagle:library:420" deviceset="R-US_" device="R0603" package3d_urn="urn:adsk.eagle:package:6240565/1" value="3.3k"/>
 <part name="C1" library="adafruit" library_urn="urn:adsk.eagle:library:420" deviceset="C-US" device="C0603" package3d_urn="urn:adsk.eagle:package:6240338/1" value="0.1µF"/>
@@
 <part name="FRAME5" library="frames" library_urn="urn:adsk.eagle:library:229" deviceset="TABL_L" device="" value="Null Value"/>
 <part name="FRAME4" library="frames" library_urn="urn:adsk.eagle:library:229" deviceset="TABL_L" device="" value="Null Value"/>
-<part name="R19" library="adafruit" library_urn="urn:adsk.eagle:library:420" deviceset="R-US_" device="R1206" package3d_urn="urn:adsk.eagle:package:6240569/1" value="0.010Ω"/>
+<part name="R19" library="adafruit" library_urn="urn:adsk.eagle:library:420" deviceset="R-US_" device="R1206" package3d_urn="urn:adsk.eagle:package:6240569/1" value="0.003Ω"/>
 <part name="R15" library="adafruit" library_urn="urn:adsk.eagle:library:420" deviceset="R-US_" device="R0603" package3d_urn="urn:adsk.eagle:package:6240565/1" value="3.3k"/>
 <part name="C11" library="adafruit" library_urn="urn:adsk.eagle:library:420" deviceset="C-US" device="C0603" package3d_urn="urn:adsk.eagle:package:6240338/1" value="100nF"/>
@@
 <part name="C34" library="adafruit" library_urn="urn:adsk.eagle:library:420" deviceset="C-US" device="C0603" package3d_urn="urn:adsk.eagle:package:6240338/1" value="0.1 mf"/>
 <part name="C32" library="adafruit" library_urn="urn:adsk.eagle:library:420" deviceset="C-US" device="C0603" package3d_urn="urn:adsk.eagle:package:6240338/1" value="270nf "/>
-<part name="R26" library="adafruit" library_urn="urn:adsk.eagle:library:420" deviceset="R-US_" device="R1206" package3d_urn="urn:adsk.eagle:package:6240569/1" value="0.005Ω 1%"/>
+<part name="R26" library="rcl" library_urn="urn:adsk.eagle:library:334" deviceset="R-US_" device="R2512" package3d_urn="urn:adsk.eagle:package:23545/2" value="0.8Ω 1%"/>
 <part name="R23" library="adafruit" library_urn="urn:adsk.eagle:library:420" deviceset="R-US_" device="R0603" package3d_urn="urn:adsk.eagle:package:6240565/1" value="3.3kΩ 1%"/>
 <part name="C23" library="adafruit" library_urn="urn:adsk.eagle:library:420" deviceset="C-US" device="C0603" package3d_urn="urn:adsk.eagle:package:6240338/1" value="0.1µF"/>
@@
 <part name="U6" library="Opamp1" deviceset="LM2904ITPX/NOPB" device=""/>
 <part name="GND58" library="supply1" library_urn="urn:adsk.eagle:library:371" deviceset="GND" device=""/>
-<part name="R25" library="adafruit" library_urn="urn:adsk.eagle:library:420" deviceset="R-US_" device="R1206" package3d_urn="urn:adsk.eagle:package:6240569/1" value="0.005Ω 1%"/>
 <part name="C27" library="adafruit" library_urn="urn:adsk.eagle:library:420" deviceset="C-US" device="050-050X075" package3d_urn="urn:adsk.eagle:package:6240360/1" value="220µF"/>
 <part name="GND59" library="SparkFun-PowerSymbols" deviceset="GND" device=""/>
@@
 <part name="J12" library="SparkFun-Connectors" deviceset="CONN_06" device="SILK_FEMALE_PTH"/>
 <part name="J13" library="SparkFun-Connectors" deviceset="CONN_06" device="SILK_FEMALE_PTH"/>
+<part name="R67" library="rcl" library_urn="urn:adsk.eagle:library:334" deviceset="R-US_" device="R2512" package3d_urn="urn:adsk.eagle:package:23545/2" value="0.8Ω 1%"/>
 </parts>
 <sheets>
@@
 <attribute name="VALUE" x="-66.04" y="20.32" size="1.778" layer="96"/>
 </instance>
-<instance part="R25" gate="G$1" x="-88.9" y="-12.7" smashed="yes">
-<attribute name="NAME" x="-92.71" y="-11.2014" size="1.778" layer="95"/>
-<attribute name="VALUE" x="-92.71" y="-16.002" size="1.778" layer="96"/>
-</instance>
 <instance part="C27" gate="G$1" x="-43.18" y="-20.32" smashed="yes">
 <attribute name="NAME" x="-42.164" y="-19.685" size="1.778" layer="95"/>
@@
 <attribute name="NAME" x="141.3256" y="-75.3872" size="1.778" layer="95" ratio="10" rot="SR0"/>
 </instance>
+<instance part="R67" gate="G$1" x="-88.9" y="-12.7" smashed="yes">
+<attribute name="NAME" x="-92.71" y="-11.2014" size="1.778" layer="95"/>
+<attribute name="VALUE" x="-92.71" y="-16.002" size="1.778" layer="96"/>
+</instance>
 </instances>
 <busses>
@@
 <pinref part="C27" gate="G$1" pin="1"/>
 <wire x1="-43.18" y1="-12.7" x2="-43.18" y2="-17.78" width="0.1524" layer="91"/>
-<pinref part="R25" gate="G$1" pin="2"/>
 <wire x1="-83.82" y1="-12.7" x2="-71.12" y2="-12.7" width="0.1524" layer="91"/>
 <wire x1="-71.12" y1="-12.7" x2="-43.18" y2="-12.7" width="0.1524" layer="91"/>
@@
 <wire x1="-43.18" y1="-12.7" x2="-17.78" y2="-12.7" width="0.1524" layer="91"/>
 <junction x="-43.18" y="-12.7"/>
+<pinref part="R67" gate="G$1" pin="2"/>
 </segment>
 <segment>
@@
 <wire x1="-116.84" y1="-12.7" x2="-121.7676" y2="-12.7" width="0.1524" layer="91"/>
 <junction x="-116.84" y="-12.7"/>
-<pinref part="R25" gate="G$1" pin="1"/>
 <wire x1="-93.98" y1="-12.7" x2="-104.14" y2="-12.7" width="0.1524" layer="91"/>
 <pinref part="U6" gate="A" pin="IN+_2"/>
@@
 <junction x="-104.14" y="-12.7"/>
 <label x="-68.58" y="5.08" size="1.778" layer="95"/>
+<pinref part="R67" gate="G$1" pin="1"/>
 </segment>
 </net>
@@
 packages will not be understood (or retained) with this version.
 </note>
+<note version="8.4" severity="warning">
+Since Version 8.4, EAGLE supports properties for SPICE simulation.
+Probes in schematics and SPICE mapping objects found in parts and library devices
+will not be understood with this version. Update EAGLE to the latest version
+for full support of SPICE simulation.
+</note>
 </compatibility>

Commit message: Resistor changes
3 resistors changed from 0.005 to 0.003
Parts:
- R11, R12, R18: value 0.005 -> 0.003
Changed lines of the file:
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@@
 <setting verticaltext="up"/>
 </settings>
-<grid distance="0.05" unitdist="inch" unit="inch" style="lines" multiple="1" display="yes" altdistance="0.01" altunitdist="inch" altunit="inch"/>
+<grid distance="0.1" unitdist="inch" unit="inch" style="lines" multiple="1" display="no" altdistance="0.01" altunitdist="inch" altunit="inch"/>
 <layers>
 <layer number="1" name="Top" color="4" fill="1" visible="no" active="no"/>
@@
 <part name="U3" library="Opamp1" deviceset="LM2904ITPX/NOPB" device=""/>
 <part name="GND26" library="supply1" library_urn="urn:adsk.eagle:library:371" deviceset="GND" device=""/>
-<part name="R12" library="adafruit" library_urn="urn:adsk.eagle:library:420" deviceset="R-US_" device="R1206" package3d_urn="urn:adsk.eagle:package:6240569/1" value="0.005"/>
+<part name="R12" library="adafruit" library_urn="urn:adsk.eagle:library:420" deviceset="R-US_" device="R1206" package3d_urn="urn:adsk.eagle:package:6240569/1" value="0.003"/>
 <part name="C8" library="adafruit" library_urn="urn:adsk.eagle:library:420" deviceset="C-US" device="050-050X075" package3d_urn="urn:adsk.eagle:package:6240360/1" value="220µF"/>
 <part name="GND29" library="SparkFun-PowerSymbols" deviceset="GND" device=""/>
@@
 <part name="U5" library="Opamp1" deviceset="LM2904ITPX/NOPB" device=""/>
 <part name="GND34" library="supply1" library_urn="urn:adsk.eagle:library:371" deviceset="GND" device=""/>
-<part name="R18" library="adafruit" library_urn="urn:adsk.eagle:library:420" deviceset="R-US_" device="R1206" package3d_urn="urn:adsk.eagle:package:6240569/1" value="0.005"/>
+<part name="R18" library="adafruit" library_urn="urn:adsk.eagle:library:420" deviceset="R-US_" device="R1206" package3d_urn="urn:adsk.eagle:package:6240569/1" value="0.003"/>
 <part name="C16" library="adafruit" library_urn="urn:adsk.eagle:library:420" deviceset="C-US" device="050-050X075" package3d_urn="urn:adsk.eagle:package:6240360/1" value="220µF"/>
 <part name="GND35" library="SparkFun-PowerSymbols" deviceset="GND" device=""/>
@@
 <part name="U2" library="Opamp1" deviceset="LM2904ITPX/NOPB" device=""/>
 <part name="GND40" library="supply1" library_urn="urn:adsk.eagle:library:371" deviceset="GND" device=""/>
-<part name="R11" library="adafruit" library_urn="urn:adsk.eagle:library:420" deviceset="R-US_" device="R1206" package3d_urn="urn:adsk.eagle:package:6240569/1" value="0.005"/>
+<part name="R11" library="adafruit" library_urn="urn:adsk.eagle:library:420" deviceset="R-US_" device="R1206" package3d_urn="urn:adsk.eagle:package:6240569/1" value="0.003"/>
 <part name="C7" library="adafruit" library_urn="urn:adsk.eagle:library:420" deviceset="C-US" device="050-050X075" package3d_urn="urn:adsk.eagle:package:6240360/1" value="220µF"/>
 <part name="GND41" library="SparkFun-PowerSymbols" deviceset="GND" device=""/>

Commit message: Resistor changes
Changed Resistor Power outputs to 0.001
Parts:
- R26, R67: value 0.8Ω 1% -> 0.001Ω 1%
Changed lines of the file:
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@@
 <part name="C34" library="adafruit" library_urn="urn:adsk.eagle:library:420" deviceset="C-US" device="C0603" package3d_urn="urn:adsk.eagle:package:6240338/1" value="0.1 mf"/>
 <part name="C32" library="adafruit" library_urn="urn:adsk.eagle:library:420" deviceset="C-US" device="C0603" package3d_urn="urn:adsk.eagle:package:6240338/1" value="270nf "/>
-<part name="R26" library="rcl" library_urn="urn:adsk.eagle:library:334" deviceset="R-US_" device="R2512" package3d_urn="urn:adsk.eagle:package:23545/2" value="0.8Ω 1%"/>
+<part name="R26" library="rcl" library_urn="urn:adsk.eagle:library:334" deviceset="R-US_" device="R2512" package3d_urn="urn:adsk.eagle:package:23545/2" value="0.001Ω 1%"/>
 <part name="R23" library="adafruit" library_urn="urn:adsk.eagle:library:420" deviceset="R-US_" device="R0603" package3d_urn="urn:adsk.eagle:package:6240565/1" value="3.3kΩ 1%"/>
 <part name="C23" library="adafruit" library_urn="urn:adsk.eagle:library:420" deviceset="C-US" device="C0603" package3d_urn="urn:adsk.eagle:package:6240338/1" value="0.1µF"/>
@@
 <part name="J12" library="SparkFun-Connectors" deviceset="CONN_06" device="SILK_FEMALE_PTH"/>
 <part name="J13" library="SparkFun-Connectors" deviceset="CONN_06" device="SILK_FEMALE_PTH"/>
-<part name="R67" library="rcl" library_urn="urn:adsk.eagle:library:334" deviceset="R-US_" device="R2512" package3d_urn="urn:adsk.eagle:package:23545/2" value="0.8Ω 1%"/>
+<part name="R67" library="rcl" library_urn="urn:adsk.eagle:library:334" deviceset="R-US_" device="R2512" package3d_urn="urn:adsk.eagle:package:23545/2" value="0.001Ω 1%"/>
 </parts>
 <sheets>

Commit message: Capacitor typo
Changed the C34 package to uf rather than mf
Parts:
- C34: value 0.1 mf -> 0.1 uf
Changed lines of the file:
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@@
 <part name="C29" library="adafruit" library_urn="urn:adsk.eagle:library:420" deviceset="C-US" device="C1206" package3d_urn="urn:adsk.eagle:package:6240335/1" value="22uF"/>
 <part name="C31" library="adafruit" library_urn="urn:adsk.eagle:library:420" deviceset="C-US" device="C1206" package3d_urn="urn:adsk.eagle:package:6240335/1" value="1.5nf"/>
-<part name="C34" library="adafruit" library_urn="urn:adsk.eagle:library:420" deviceset="C-US" device="C0603" package3d_urn="urn:adsk.eagle:package:6240338/1" value="0.1 mf"/>
+<part name="C34" library="adafruit" library_urn="urn:adsk.eagle:library:420" deviceset="C-US" device="C0603" package3d_urn="urn:adsk.eagle:package:6240338/1" value="0.1 uf"/>
 <part name="C32" library="adafruit" library_urn="urn:adsk.eagle:library:420" deviceset="C-US" device="C0603" package3d_urn="urn:adsk.eagle:package:6240338/1" value="270nf "/>
 <part name="R26" library="rcl" library_urn="urn:adsk.eagle:library:334" deviceset="R-US_" device="R2512" package3d_urn="urn:adsk.eagle:package:23545/2" value="0.001Ω 1%"/>

Commit message: Compasitors
Changed the capacitors to the correct 3.5mm pitch.
Parts:
- C10, C16, C17, C18, C27, C28, C7, C8, C9: device adafruit:C-US050-050X075 -> Rapid_Prototype_Schematic:ADAFRUIT_C-US3.5MMCAP
Changed lines of the file:
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@@
 <part name="C2" library="adafruit" library_urn="urn:adsk.eagle:library:420" deviceset="C-US" device="C0603" package3d_urn="urn:adsk.eagle:package:6240338/1" value="0.1µF"/>
 <part name="C4" library="adafruit" library_urn="urn:adsk.eagle:library:420" deviceset="C-US" device="C0603" package3d_urn="urn:adsk.eagle:package:6240338/1" value="1µF"/>
-<part name="C10" library="adafruit" library_urn="urn:adsk.eagle:library:420" deviceset="C-US" device="050-050X075" package3d_urn="urn:adsk.eagle:package:6240360/1" value="220µF"/>
+<part name="C10" library="Rapid_Prototype_Schematic" deviceset="ADAFRUIT_C-US" device="3.5MMCAP" value="220µF"/>
 <part name="GND25" library="SparkFun-PowerSymbols" deviceset="GND" device=""/>
 <part name="GND27" library="SparkFun-PowerSymbols" deviceset="GND" device=""/>
@@
 <part name="GND26" library="supply1" library_urn="urn:adsk.eagle:library:371" deviceset="GND" device=""/>
 <part name="R12" library="adafruit" library_urn="urn:adsk.eagle:library:420" deviceset="R-US_" device="R1206" package3d_urn="urn:adsk.eagle:package:6240569/1" value="0.003"/>
-<part name="C8" library="adafruit" library_urn="urn:adsk.eagle:library:420" deviceset="C-US" device="050-050X075" package3d_urn="urn:adsk.eagle:package:6240360/1" value="220µF"/>
+<part name="C8" library="Rapid_Prototype_Schematic" deviceset="ADAFRUIT_C-US" device="3.5MMCAP" value="220µF"/>
 <part name="GND29" library="SparkFun-PowerSymbols" deviceset="GND" device=""/>
 <part name="R10" library="adafruit" library_urn="urn:adsk.eagle:library:420" deviceset="R-US_" device="R0603" package3d_urn="urn:adsk.eagle:package:6240565/1" value="3.3k"/>
@@
 <part name="C12" library="adafruit" library_urn="urn:adsk.eagle:library:420" deviceset="C-US" device="C0603" package3d_urn="urn:adsk.eagle:package:6240338/1" value="0.1µF"/>
 <part name="C14" library="adafruit" library_urn="urn:adsk.eagle:library:420" deviceset="C-US" device="C0603" package3d_urn="urn:adsk.eagle:package:6240338/1" value="1µF"/>
-<part name="C18" library="adafruit" library_urn="urn:adsk.eagle:library:420" deviceset="C-US" device="050-050X075" package3d_urn="urn:adsk.eagle:package:6240360/1" value="220µF"/>
+<part name="C18" library="Rapid_Prototype_Schematic" deviceset="ADAFRUIT_C-US" device="3.5MMCAP" value="220µF"/>
 <part name="GND30" library="SparkFun-PowerSymbols" deviceset="GND" device=""/>
 <part name="GND32" library="SparkFun-PowerSymbols" deviceset="GND" device=""/>
@@
 <part name="GND34" library="supply1" library_urn="urn:adsk.eagle:library:371" deviceset="GND" device=""/>
 <part name="R18" library="adafruit" library_urn="urn:adsk.eagle:library:420" deviceset="R-US_" device="R1206" package3d_urn="urn:adsk.eagle:package:6240569/1" value="0.003"/>
-<part name="C16" library="adafruit" library_urn="urn:adsk.eagle:library:420" deviceset="C-US" device="050-050X075" package3d_urn="urn:adsk.eagle:package:6240360/1" value="220µF"/>
+<part name="C16" library="Rapid_Prototype_Schematic" deviceset="ADAFRUIT_C-US" device="3.5MMCAP" value="220µF"/>
 <part name="GND35" library="SparkFun-PowerSymbols" deviceset="GND" device=""/>
 <part name="R17" library="adafruit" library_urn="urn:adsk.eagle:library:420" deviceset="R-US_" device="R0603" package3d_urn="urn:adsk.eagle:package:6240565/1" value="3.3k"/>
@@
 <part name="C1" library="adafruit" library_urn="urn:adsk.eagle:library:420" deviceset="C-US" device="C0603" package3d_urn="urn:adsk.eagle:package:6240338/1" value="0.1µF"/>
 <part name="C3" library="adafruit" library_urn="urn:adsk.eagle:library:420" deviceset="C-US" device="C0603" package3d_urn="urn:adsk.eagle:package:6240338/1" value="1µF"/>
-<part name="C9" library="adafruit" library_urn="urn:adsk.eagle:library:420" deviceset="C-US" device="050-050X075" package3d_urn="urn:adsk.eagle:package:6240360/1" value="220µF"/>
+<part name="C9" library="Rapid_Prototype_Schematic" deviceset="ADAFRUIT_C-US" device="3.5MMCAP" value="220µF"/>
 <part name="GND37" library="SparkFun-PowerSymbols" deviceset="GND" device=""/>
 <part name="GND38" library="SparkFun-PowerSymbols" deviceset="GND" device=""/>
@@
 <part name="GND40" library="supply1" library_urn="urn:adsk.eagle:library:371" deviceset="GND" device=""/>
 <part name="R11" library="adafruit" library_urn="urn:adsk.eagle:library:420" deviceset="R-US_" device="R1206" package3d_urn="urn:adsk.eagle:package:6240569/1" value="0.003"/>
-<part name="C7" library="adafruit" library_urn="urn:adsk.eagle:library:420" deviceset="C-US" device="050-050X075" package3d_urn="urn:adsk.eagle:package:6240360/1" value="220µF"/>
+<part name="C7" library="Rapid_Prototype_Schematic" deviceset="ADAFRUIT_C-US" device="3.5MMCAP" value="220µF"/>
 <part name="GND41" library="SparkFun-PowerSymbols" deviceset="GND" device=""/>
 <part name="R9" library="adafruit" library_urn="urn:adsk.eagle:library:420" deviceset="R-US_" device="R0603" package3d_urn="urn:adsk.eagle:package:6240565/1" value="3.3k"/>
@@
 <part name="C11" library="adafruit" library_urn="urn:adsk.eagle:library:420" deviceset="C-US" device="C0603" package3d_urn="urn:adsk.eagle:package:6240338/1" value="100nF"/>
 <part name="C13" library="adafruit" library_urn="urn:adsk.eagle:library:420" deviceset="C-US" device="C0805" package3d_urn="urn:adsk.eagle:package:6240337/1" value="1uF"/>
-<part name="C17" library="adafruit" library_urn="urn:adsk.eagle:library:420" deviceset="C-US" device="050-050X075" package3d_urn="urn:adsk.eagle:package:6240360/1" value="220uF"/>
+<part name="C17" library="Rapid_Prototype_Schematic" deviceset="ADAFRUIT_C-US" device="3.5MMCAP" value="220uF"/>
 <part name="GND63" library="SparkFun-PowerSymbols" deviceset="GND" device=""/>
 <part name="GND64" library="SparkFun-PowerSymbols" deviceset="GND" device=""/>
@@
 <part name="C23" library="adafruit" library_urn="urn:adsk.eagle:library:420" deviceset="C-US" device="C0603" package3d_urn="urn:adsk.eagle:package:6240338/1" value="0.1µF"/>
 <part name="C24" library="adafruit" library_urn="urn:adsk.eagle:library:420" deviceset="C-US" device="C0603" package3d_urn="urn:adsk.eagle:package:6240338/1" value="1µF"/>
-<part name="C28" library="adafruit" library_urn="urn:adsk.eagle:library:420" deviceset="C-US" device="050-050X075" package3d_urn="urn:adsk.eagle:package:6240360/1" value="220µF"/>
+<part name="C28" library="Rapid_Prototype_Schematic" deviceset="ADAFRUIT_C-US" device="3.5MMCAP" value="220µF"/>
 <part name="GND54" library="SparkFun-PowerSymbols" deviceset="GND" device=""/>
 <part name="GND56" library="SparkFun-PowerSymbols" deviceset="GND" device=""/>
@@
 <part name="U6" library="Opamp1" deviceset="LM2904ITPX/NOPB" device=""/>
 <part name="GND58" library="supply1" library_urn="urn:adsk.eagle:library:371" deviceset="GND" device=""/>
-<part name="C27" library="adafruit" library_urn="urn:adsk.eagle:library:420" deviceset="C-US" device="050-050X075" package3d_urn="urn:adsk.eagle:package:6240360/1" value="220µF"/>
+<part name="C27" library="Rapid_Prototype_Schematic" deviceset="ADAFRUIT_C-US" device="3.5MMCAP" value="220µF"/>
 <part name="GND59" library="SparkFun-PowerSymbols" deviceset="GND" device=""/>
 <part name="R24" library="adafruit" library_urn="urn:adsk.eagle:library:420" deviceset="R-US_" device="R0603" package3d_urn="urn:adsk.eagle:package:6240565/1" value="3.3kΩ 1%"/>

Commit message: Capacitor Size Changes
Replaced and made capacitors smaller
Parts:
- C19, C25, C26, C35, C36, C37, C38, C39, C40, C41: value 1µF -> 1.0uF; device adafruit:C-USC0805 -> SparkFun-Capacitors:1.0UF-0603-16V-10%-X7R
- C24: value 1µF -> 1.0uF; device adafruit:C-USC0603 -> SparkFun-Capacitors:1.0UF-0603-16V-10%-X7R
Other:
- moved on the sheet: C19, C24, C25, C26, C35, C36, C37, C38, C39, C40, C41
