File: Rapid_Prototype_Schematic.sch (EAGLE design)
At the start: 177 parts, among them IC2 SI4459ADY-T1-GE3, IC8 SI4485DY-T1-GE3, J1 XT60-M, J10 XT60-M, J2 XT60-M, J3 Vertical Qwiic Connector, J4 UJ2-MIBH-2-SMT-TR-67, J5 XT60-M, J6 XT60-M, J7 XT60-M, J8 XT60-M, J9 XT60-M, Q1 LTV-8141S, Q10 SI4435DDY, Q11 DMN65D8LFB-7, Q12 SI4435DDY, Q13 DMN65D8LFB-7, Q14 SI4435DDY, Q15 DMN65D8LFB-7, Q16 2N7002PW, Q2 2N7002PW, Q3 DMN65D8LFB-7, Q4 SI4435DDY, Q5 DMN65D8LFB-7, Q6 SI4435DDY, Q7 DMN65D8LFB-7, Q8 SI4435DDY, Q9 DMN65D8LFB-7, U1 LM35DM, U2 LM2904ITPX/NOPB, U3 LM2904ITPX/NOPB, U4 LM2904ITPX/NOPB, U5 LM2904ITPX/NOPB, U6 LM2904ITPX/NOPB, U7 TLV1117LV33DCYR, U8 LT1374IS8-5PBF

Commit message: Changing units in Schematic
Changed C11 and C30 from 100nF to 0.1 uF, this allows us to order those parts without needing quantity change
Parts:
- C11: value 100nF -> 0.1uF
- C30: value 100nf -> 0.1uF
Changed lines of the file:
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@@
 <part name="R19" library="adafruit" library_urn="urn:adsk.eagle:library:420" deviceset="R-US_" device="R1206" package3d_urn="urn:adsk.eagle:package:6240569/1" value="0.003Ω"/>
 <part name="R15" library="adafruit" library_urn="urn:adsk.eagle:library:420" deviceset="R-US_" device="R0603" package3d_urn="urn:adsk.eagle:package:6240565/1" value="3.3k"/>
-<part name="C11" library="adafruit" library_urn="urn:adsk.eagle:library:420" deviceset="C-US" device="C0603" package3d_urn="urn:adsk.eagle:package:6240338/1" value="100nF"/>
+<part name="C11" library="adafruit" library_urn="urn:adsk.eagle:library:420" deviceset="C-US" device="C0603" package3d_urn="urn:adsk.eagle:package:6240338/1" value="0.1uF"/>
 <part name="C13" library="adafruit" library_urn="urn:adsk.eagle:library:420" deviceset="C-US" device="C0805" package3d_urn="urn:adsk.eagle:package:6240337/1" value="1uF"/>
 <part name="C17" library="Rapid_Prototype_Schematic" deviceset="ADAFRUIT_C-US" device="3.5MMCAP" value="220uF"/>
@@
 <part name="GND75" library="supply1" library_urn="urn:adsk.eagle:library:371" deviceset="GND" device=""/>
 <part name="GND76" library="supply1" library_urn="urn:adsk.eagle:library:371" deviceset="GND" device=""/>
-<part name="C30" library="adafruit" library_urn="urn:adsk.eagle:library:420" deviceset="C-US" device="C0603" package3d_urn="urn:adsk.eagle:package:6240338/1" value="100nf"/>
+<part name="C30" library="adafruit" library_urn="urn:adsk.eagle:library:420" deviceset="C-US" device="C0603" package3d_urn="urn:adsk.eagle:package:6240338/1" value="0.1uF"/>
 <part name="C33" library="adafruit" library_urn="urn:adsk.eagle:library:420" deviceset="C-US" device="C0603" package3d_urn="urn:adsk.eagle:package:6240338/1" value="10uf"/>
 <part name="CR1" library="Diode1" deviceset="BZT585B16T-7" device="SOD523-M"/>
