File: Rapid_Prototype_Schematic.brd (EAGLE design)
At the start: 142 x 95 mm, 177 parts, among them IC2 SI4459ADY-T1-GE3, IC8 SI4485DY-T1-GE3, J1 XT60-M, J10 XT60-M, J2 XT60-M, J3 Vertical Qwiic Connector, J4 UJ2-MIBH-2-SMT-TR-67, J5 XT60-M, J6 XT60-M, J7 XT60-M, J8 XT60-M, J9 XT60-M, Q1 LTV-8141S, Q10 SI4435DDY, Q11 DMN65D8LFB-7, Q12 SI4435DDY, Q13 DMN65D8LFB-7, Q14 SI4435DDY, Q15 DMN65D8LFB-7, Q16 2N7002PW, Q2 2N7002PW, Q3 DMN65D8LFB-7, Q4 SI4435DDY, Q5 DMN65D8LFB-7, Q6 SI4435DDY, Q7 DMN65D8LFB-7, Q8 SI4435DDY, Q9 DMN65D8LFB-7, U1 LM35DM, U2 LM2904ITPX/NOPB, U3 LM2904ITPX/NOPB, U4 LM2904ITPX/NOPB, U5 LM2904ITPX/NOPB, U6 LM2904ITPX/NOPB, U7 TLV1117LV33DCYR, U8 LT1374IS8-5PBF

Commit message: Resistor changes
3 resistors changed from 0.005 to 0.003
Parts:
- R11, R12, R18: value 0.005 -> 0.003
Changed lines of the file:
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@@
 <attribute name="VALUE" x="46.482" y="88.138" size="1.27" layer="27" rot="R270"/>
 </element>
-<element name="R11" library="adafruit" library_urn="urn:adsk.eagle:library:420" package="R1206" package3d_urn="urn:adsk.eagle:package:6240569/1" value="0.005" x="74.93" y="72.39" smashed="yes" rot="R270">
+<element name="R11" library="adafruit" library_urn="urn:adsk.eagle:library:420" package="R1206" package3d_urn="urn:adsk.eagle:package:6240569/1" value="0.003" x="74.93" y="72.39" smashed="yes" rot="R270">
 <attribute name="NAME" x="76.073" y="73.787" size="0.8128" layer="25" rot="R270"/>
 <attribute name="VALUE" x="72.517" y="73.787" size="1.27" layer="27" rot="R270"/>
 </element>
-<element name="R12" library="adafruit" library_urn="urn:adsk.eagle:library:420" package="R1206" package3d_urn="urn:adsk.eagle:package:6240569/1" value="0.005" x="85.09" y="72.39" smashed="yes" rot="R270">
+<element name="R12" library="adafruit" library_urn="urn:adsk.eagle:library:420" package="R1206" package3d_urn="urn:adsk.eagle:package:6240569/1" value="0.003" x="85.09" y="72.39" smashed="yes" rot="R270">
 <attribute name="NAME" x="86.233" y="73.787" size="0.8128" layer="25" rot="R270"/>
 <attribute name="VALUE" x="82.677" y="73.787" size="1.27" layer="27" rot="R270"/>
@@
 <attribute name="VALUE" x="45.847" y="86.614" size="1.27" layer="27" rot="R90"/>
 </element>
-<element name="R18" library="adafruit" library_urn="urn:adsk.eagle:library:420" package="R1206" package3d_urn="urn:adsk.eagle:package:6240569/1" value="0.005" x="60.96" y="72.39" smashed="yes" rot="R270">
+<element name="R18" library="adafruit" library_urn="urn:adsk.eagle:library:420" package="R1206" package3d_urn="urn:adsk.eagle:package:6240569/1" value="0.003" x="60.96" y="72.39" smashed="yes" rot="R270">
 <attribute name="NAME" x="62.103" y="73.787" size="0.8128" layer="25" rot="R270"/>
 <attribute name="VALUE" x="58.547" y="73.787" size="1.27" layer="27" rot="R270"/>
